Commit message: Created Gazebo_Cotrol

File: description/robot_core.xacro (robot description, xacro)
@@ -41,4 +41,7 @@
     </xacro:inertial_box>
 </link>
+<gazebo reference="chassis">
+    <material>Gazebo/Orange</material>
+</gazebo>
     <!-- LEFT WHEEL -->
 <joint name="left_wheel_joint" type="continuous">
@@ -64,4 +67,7 @@
     </xacro:inertial_cylinder>
 </link>
+<gazebo reference="left_wheel">
+    <material>Gazebo/Blue</material>
+</gazebo>
     <!-- RIGHT WHEEL -->
 <joint name="right_wheel_joint" type="continuous">
@@ -87,4 +93,7 @@
     </xacro:inertial_cylinder>
 </link>
+<gazebo reference="right_wheel">
+    <material>Gazebo/Blue</material>
+</gazebo>
 <!-- CASTER WHEEL -->
 <joint name="caster_wheel_joint" type="fixed">
@@ -109,3 +118,8 @@
     </xacro:inertial_sphere>
 </link>
+<gazebo reference="caster_wheel">
+    <material>Gazebo/Black</material>
+    <mu1 value="0.001"/>
+    <mu2 value="0.001"/>
+</gazebo>
 </robot>

Commit message: slam toolbox added

File: description/robot_core.xacro (robot description, xacro)
@@ -14,4 +14,7 @@
     <color rgba="0 0 0 1"/>
 </material>
+<material name="red">
+    <color rgba="1 0 0 1"/>
+</material>
 <link name="base_link">
 </link>
@@ -22,4 +25,12 @@
     <origin xyz="-0.1 0 0"/>
 </joint>
+    <!--BASE FOOTPRINT-->
+<joint name="base_footprint_joint" type="fixed">
+    <parent link="base_link"/>
+    <child link="base_footprint"/>
+    <origin xyz="0 0 0" rpy ="0 0 0" />
+</joint>
+<link name="base_footprint">
+</link>
     <!--CHASSIS-->
 <link name="chassis">
@@ -42,5 +53,5 @@
 </link>
 <gazebo reference="chassis">
-    <material>Gazebo/Orange</material>
+    <material>Gazebo/White</material>
 </gazebo>
     <!-- LEFT WHEEL -->
